File: altitude-ctrl-1.kicad_pcb (KiCad board)
At the start: 2 copper layers, 93 parts, among them J1 Conn_01x02, J10 Conn_01x02, J2 Conn_01x02, J3 Conn_01x05, J4 TC2030, J5 Conn_01x04_Pin, J6 Conn_01x02, J7 Conn_01x05, J8 Conn_01x05, J9 Conn_01x02, SW1 SW_Push, SW2 SW_SPST, SW3 SW_Push, SW4 SW_SPST, SW5 SW_Push, U1 HT753-1, U2 ULN2003A, U3 LM73100, U4 LM73100, U5 MAX6675, U6 STM32F103C8Tx, U7 SN65HVD230, Y1 8M

Commit message: pcb: add board outline and mnt holes
Parts:
- moved H5 193.2 mm to (213.8, 34.5)
- moved H4 180.3 mm to (213.8, 99.5)
- moved J7 143.7 mm to (134.8, 57.3), turned to -90 degrees
- moved H6 131.8 mm to (146.8, 34.5)
- moved D17 124.2 mm to (142.1, 72.0), turned to 0 degrees
- moved D15 122.9 mm to (142.1, 70.0), turned to 0 degrees
- moved D13 121.6 mm to (142.1, 68.0), turned to 0 degrees
- moved D11 120.4 mm to (142.1, 66.1), turned to 0 degrees
- moved SW4 106.2 mm to (134.8, 31.9), turned to -90 degrees
- moved J8 101.7 mm to (134.8, 82.7), turned to -90 degrees
- moved SW2 91.0 mm to (134.8, 42.1), turned to -90 degrees
- moved D18 82.5 mm to (141.9, 95.2), turned to 0 degrees
- moved D16 80.9 mm to (141.9, 93.2), turned to 0 degrees
- moved D14 79.4 mm to (141.9, 91.2), turned to 0 degrees
- moved D12 77.9 mm to (141.9, 89.2), turned to 0 degrees
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Other:
- board outline added: 90 x 90 mm
